Commit message: 記述追加

File: mikata_arm_moveit/config/mikata_arm.ros2_control.xacro (robot description, xacro)
@@ -2,5 +2,5 @@
 <robot xmlns:xacro="http://www.ros.org/wiki/xacro">
     <xacro:macro name="mikata_arm_ros2_control" params="name initial_positions_file">
-        <xacro:property name="initial_positions" value="${load_yaml(initial_positions_file)['initial_positions']}"/>
+      <xacro:property name="initial_positions" value="${xacro.load_yaml(initial_positions_file)['initial_positions']}"/>
         <ros2_control name="${name}" type="system">
             <hardware>
@@ -57,4 +57,10 @@
                 <state_interface name="velocity"/>
             </joint>
+            <joint name="gripper_sub2">
+                <state_interface name="position">
+                  <param name="initial_value">${initial_positions['gripper_sub2']}</param>
+                </state_interface>
+                <state_interface name="velocity"/>
+            </joint>
         </ros2_control>
     </xacro:macro>
