Commit message: joint名を変更

File: mikata_arm_bringup/config/mikata_arm.ros2_control.xacro (robot description, xacro)
@@ -43,8 +43,8 @@
                 <state_interface name="velocity"/>
             </joint>
-            <joint name="gripper_joint">
+            <joint name="joint6">
                 <command_interface name="position"/>
                 <state_interface name="position">
-                  <param name="initial_value">${initial_positions['gripper_joint']}</param>
+                  <param name="initial_value">${initial_positions['joint6']}</param>
                 </state_interface>
                 <state_interface name="velocity"/>

File: mikata_arm_description/urdf/mikata_arm.xacro (robot description, xacro)
@@ -215,5 +215,5 @@
     </collision>
   </link>
-  <joint name="gripper_joint" type="revolute">
+  <joint name="joint6" type="revolute">
     <origin xyz="0.045 2.1e-05 0.0" rpy="0.0 0.0 0.0"/>
     <axis xyz="1 0 0"/>
