Commit message: ハードウェア接続の設定を更新し、初期位置の定義を整理

File: mikata_arm_bringup/config/mikata_arm.system.urdf.xacro (robot description, xacro)
@@ -3,6 +3,19 @@
   <xacro:arg name="prefix" default="" />
   <xacro:arg name="initial_positions_file" default="$(find mikata_arm_bringup)/config/initial_positions.yaml" />
-  <xacro:include filename="$(find mikata_arm_description)/urdf/mikata_arm.urdf.xacro" />
-  <xacro:include filename="$(find mikata_arm_bringup)/config/mikata_arm.ros2_control.xacro" />
-  <xacro:mikata_arm_ros2_control name="FakeSystem" initial_positions_file="$(arg initial_positions_file)" />
+  <!-- Include robot model only (without ros2_control) -->
+  <xacro:include filename="$(find mikata_arm_description)/urdf/mikata_arm.xacro" />
+  <xacro:include filename="$(find mikata_arm_description)/config/mikata_arm.ros2_control.xacro" />
+  <!-- Base link -->
+  <link name="$(arg prefix)base_link" />
+  <!-- Robot arm -->
+  <xacro:mikata_arm
+      prefix="$(arg prefix)"
+      parent="$(arg prefix)base_link">
+    <origin xyz="0 0 0" rpy="0 0 0" />
+  </xacro:mikata_arm>
+  <!-- Hardware interface (single definition) -->
+  <xacro:mikata_arm_ros2_control
+    name="mikata_arm"
+    prefix="$(arg prefix)"
+    initial_positions_file="$(arg initial_positions_file)" />
 </robot>

File: mikata_arm_description/config/mikata_arm.ros2_control.xacro (robot description, xacro)
@@ -1,5 +1,5 @@
 <?xml version="1.0"?>
 <robot xmlns:xacro="http://www.ros.org/wiki/xacro">
-  <xacro:macro name="mikata_arm_ros2_control" params="name">
+  <xacro:macro name="mikata_arm_ros2_control" params="name prefix:='' initial_positions_file:=''">
     <ros2_control name="${name}" type="system">
       <hardware>
@@ -7,7 +7,10 @@
         <param name="usb_port">/dev/ttyUSB0</param>
         <param name="baud_rate">1000000</param>
-        <!-- <param name="use_dummy">true</param> -->
+        <param name="use_dummy">false</param>
+        <xacro:if value="${initial_positions_file != ''}">
+          <param name="initial_positions_file">${initial_positions_file}</param>
+        </xacro:if>
       </hardware>
-      <joint name="joint1">
+      <joint name="${prefix}joint1">
         <param name="id">11</param>
         <command_interface name="position"/>
@@ -17,5 +20,5 @@
         <state_interface name="effort"/>
       </joint>
-      <joint name="joint2">
+      <joint name="${prefix}joint2">
         <param name="id">12</param>
         <command_interface name="position"/>
@@ -25,5 +28,5 @@
         <state_interface name="effort"/>
       </joint>
-      <joint name="joint3">
+      <joint name="${prefix}joint3">
         <param name="id">13</param>
         <command_interface name="position"/>
@@ -33,5 +36,5 @@
         <state_interface name="effort"/>
       </joint>
-      <joint name="joint4">
+      <joint name="${prefix}joint4">
         <param name="id">14</param>
         <command_interface name="position"/>
@@ -41,5 +44,5 @@
         <state_interface name="effort"/>
       </joint>
-      <joint name="joint5">
+      <joint name="${prefix}joint5">
         <param name="id">15</param>
         <command_interface name="position"/>
@@ -49,5 +52,5 @@
         <state_interface name="effort"/>
       </joint>
-      <joint name="joint6">
+      <joint name="${prefix}joint6">
         <param name="id">16</param>
         <command_interface name="position"/>
@@ -57,5 +60,5 @@
         <state_interface name="effort"/>
       </joint>
-      <joint name="gripper_sub1">
+      <joint name="${prefix}gripper_sub1">
         <param name="id">17</param>
         <command_interface name="position"/>

File: mikata_arm_description/urdf/mikata_arm.urdf.xacro (robot description, xacro)
@@ -5,5 +5,5 @@
   <xacro:include filename="$(find mikata_arm_description)/urdf/mikata_arm.xacro" />
   <!-- Import mikata_arm ros2_control description -->
-  <!-- <xacro:include filename="$(find mikata_arm_description)/ros2_control/mikata_arm.ros2_control.xacro" /> -->
+  <xacro:include filename="$(find mikata_arm_description)/config/mikata_arm.ros2_control.xacro" />
   <link name="$(arg prefix)base_link" />
   <xacro:mikata_arm
@@ -14,5 +14,5 @@
         rpy="0 0 0" />
   </xacro:mikata_arm>
-  <!-- <xacro:mikata_arm_ros2_control
-    name="mikata_arm" prefix="$(arg prefix)" /> -->
+  <xacro:mikata_arm_ros2_control
+    name="mikata_arm" prefix="$(arg prefix)" />
 </robot>

File: mikata_arm_description/urdf/mikata_arm.xacro (robot description, xacro)
@@ -281,5 +281,5 @@
   <joint name="gripper_sub1" type="revolute">
     <origin xyz="0.045 0.0148 -0.011" rpy="0.0 0.0 0.0"/>
-    <axis xyz="0 0 1"/>
+    <axis xyz="0 0 -1"/>
     <parent link="gripper_base"/>
     <child link="gripper_link1"/>
@@ -314,5 +314,5 @@
   <joint name="gripper_sub2" type="revolute">
     <origin xyz="0.045 -0.0172 -0.011" rpy="0.0 0.0 0.0"/>
-    <axis xyz="0 0 1"/>
+    <axis xyz="0 0 -1"/>
     <parent link="gripper_base"/>
     <child link="gripper_link2"/>
