Commit message: 一旦、URDFに仮のメッシュとしてaxis_placement_dynamixel_mikata_armのメッシュを追加

File: mikata_arm_description/urdf/mikata_arm.xacro (robot description, xacro)
@@ -1,248 +1,270 @@
-<?xml version="1.0" encoding="UTF-8"?>
+<?xml version="1.0"?>
 <robot xmlns:xacro="http://www.ros.org/wiki/xacro">
   <xacro:macro name="mikata_arm" params="prefix parent *origin">
-    <!-- Joint properties -->
-    <xacro:property name="joint_damping" value="0.5"/>
-    <xacro:property name="joint_friction" value="0.1"/>
-    <xacro:property name="joint_effort_limit" value="100.0"/>
-    <xacro:property name="joint_velocity_limit" value="3.14"/>
-    <!-- Link dimensions (approximate values for 6-axis arm) -->
-    <xacro:property name="base_height" value="0.1"/>
-    <xacro:property name="base_radius" value="0.08"/>
-    <xacro:property name="link1_length" value="0.15"/>
-    <xacro:property name="link2_length" value="0.25"/>
-    <xacro:property name="link3_length" value="0.22"/>
-    <xacro:property name="link4_length" value="0.15"/>
-    <xacro:property name="link5_length" value="0.08"/>
-    <xacro:property name="link6_length" value="0.05"/>
-    <xacro:property name="link_radius" value="0.04"/>
-    <!-- Base link attachment -->
-    <joint name="${prefix}base_joint" type="fixed">
-      <xacro:insert_block name="origin"/>
-      <parent link="${parent}"/>
-      <child link="${prefix}link_base"/>
-    </joint>
-    <!-- Base Link -->
-    <link name="${prefix}link_base">
-      <visual>
-        <origin xyz="0 0 ${base_height/2}" rpy="0 0 0"/>
-        <geometry>
-          <cylinder radius="${base_radius}" length="${base_height}"/>
-        </geometry>
-        <material name="grey">
-          <color rgba="0.5 0.5 0.5 1"/>
-        </material>
-      </visual>
-      <collision>
-        <origin xyz="0 0 ${base_height/2}" rpy="0 0 0"/>
-        <geometry>
-          <cylinder radius="${base_radius}" length="${base_height}"/>
-        </geometry>
-      </collision>
-      <inertial>
-        <origin xyz="0 0 ${base_height/2}" rpy="0 0 0"/>
-        <mass value="1.0"/>
-        <inertia ixx="0.001" ixy="0.0" ixz="0.0" iyy="0.001" iyz="0.0" izz="0.001"/>
-      </inertial>
-    </link>
-    <!-- Joint 1: Base rotation -->
-    <joint name="${prefix}joint1" type="revolute">
-      <parent link="${prefix}link_base"/>
-      <child link="${prefix}link1"/>
-      <origin xyz="0 0 ${base_height}" rpy="0 0 0"/>
-      <axis xyz="0 0 1"/>
-      <limit lower="${-pi}" upper="${pi}" effort="${joint_effort_limit}" velocity="${joint_velocity_limit}"/>
-      <dynamics damping="${joint_damping}" friction="${joint_friction}"/>
-    </joint>
-    <!-- Link 1 -->
-    <link name="${prefix}link1">
-      <visual>
-        <origin xyz="0 0 ${link1_length/2}" rpy="0 0 0"/>
-        <geometry>
-          <cylinder radius="${link_radius}" length="${link1_length}"/>
-        </geometry>
-        <material name="blue">
-          <color rgba="0.2 0.2 0.8 1"/>
-        </material>
-      </visual>
-      <collision>
-        <origin xyz="0 0 ${link1_length/2}" rpy="0 0 0"/>
-        <geometry>
-          <cylinder radius="${link_radius}" length="${link1_length}"/>
-        </geometry>
-      </collision>
-      <inertial>
-        <origin xyz="0 0 ${link1_length/2}" rpy="0 0 0"/>
-        <mass value="0.5"/>
-        <inertia ixx="0.001" ixy="0.0" ixz="0.0" iyy="0.001" iyz="0.0" izz="0.0001"/>
-      </inertial>
-    </link>
-    <!-- Joint 2: Shoulder -->
-    <joint name="${prefix}joint2" type="revolute">
-      <parent link="${prefix}link1"/>
-      <child link="${prefix}link2"/>
-      <origin xyz="0 0 ${link1_length}" rpy="0 0 0"/>
-      <axis xyz="0 1 0"/>
-      <limit lower="${-pi/2}" upper="${pi/2}" effort="${joint_effort_limit}" velocity="${joint_velocity_limit}"/>
-      <dynamics damping="${joint_damping}" friction="${joint_friction}"/>
-    </joint>
-    <!-- Link 2 -->
-    <link name="${prefix}link2">
-      <visual>
-        <origin xyz="${link2_length/2} 0 0" rpy="0 ${pi/2} 0"/>
-        <geometry>
-          <cylinder radius="${link_radius}" length="${link2_length}"/>
-        </geometry>
-        <material name="red">
-          <color rgba="0.8 0.2 0.2 1"/>
-        </material>
-      </visual>
-      <collision>
-        <origin xyz="${link2_length/2} 0 0" rpy="0 ${pi/2} 0"/>
-        <geometry>
-          <cylinder radius="${link_radius}" length="${link2_length}"/>
-        </geometry>
-      </collision>
-      <inertial>
-        <origin xyz="${link2_length/2} 0 0" rpy="0 0 0"/>
-        <mass value="0.8"/>
-        <inertia ixx="0.001" ixy="0.0" ixz="0.0" iyy="0.004" iyz="0.0" izz="0.004"/>
-      </inertial>
-    </link>
-    <!-- Joint 3: Elbow -->
-    <joint name="${prefix}joint3" type="revolute">
-      <parent link="${prefix}link2"/>
-      <child link="${prefix}link3"/>
-      <origin xyz="${link2_length} 0 0" rpy="0 0 0"/>
-      <axis xyz="0 1 0"/>
-      <limit lower="${-pi}" upper="${pi}" effort="${joint_effort_limit}" velocity="${joint_velocity_limit}"/>
-      <dynamics damping="${joint_damping}" friction="${joint_friction}"/>
-    </joint>
-    <!-- Link 3 -->
-    <link name="${prefix}link3">
-      <visual>
-        <origin xyz="${link3_length/2} 0 0" rpy="0 ${pi/2} 0"/>
-        <geometry>
-          <cylinder radius="${link_radius}" length="${link3_length}"/>
-        </geometry>
-        <material name="green">
-          <color rgba="0.2 0.8 0.2 1"/>
-        </material>
-      </visual>
-      <collision>
-        <origin xyz="${link3_length/2} 0 0" rpy="0 ${pi/2} 0"/>
-        <geometry>
-          <cylinder radius="${link_radius}" length="${link3_length}"/>
-        </geometry>
-      </collision>
-      <inertial>
-        <origin xyz="${link3_length/2} 0 0" rpy="0 0 0"/>
-        <mass value="0.6"/>
-        <inertia ixx="0.001" ixy="0.0" ixz="0.0" iyy="0.003" iyz="0.0" izz="0.003"/>
-      </inertial>
-    </link>
-    <!-- Joint 4: Wrist roll -->
-    <joint name="${prefix}joint4" type="revolute">
-      <parent link="${prefix}link3"/>
-      <child link="${prefix}link4"/>
-      <origin xyz="${link3_length} 0 0" rpy="0 0 0"/>
-      <axis xyz="1 0 0"/>
-      <limit lower="${-pi}" upper="${pi}" effort="${joint_effort_limit}" velocity="${joint_velocity_limit}"/>
-      <dynamics damping="${joint_damping}" friction="${joint_friction}"/>
-    </joint>
-    <!-- Link 4 -->
-    <link name="${prefix}link4">
-      <visual>
-        <origin xyz="${link4_length/2} 0 0" rpy="0 ${pi/2} 0"/>
-        <geometry>
-          <cylinder radius="${link_radius*0.8}" length="${link4_length}"/>
-        </geometry>
-        <material name="yellow">
-          <color rgba="0.8 0.8 0.2 1"/>
-        </material>
-      </visual>
-      <collision>
-        <origin xyz="${link4_length/2} 0 0" rpy="0 ${pi/2} 0"/>
-        <geometry>
-          <cylinder radius="${link_radius*0.8}" length="${link4_length}"/>
-        </geometry>
-      </collision>
-      <inertial>
-        <origin xyz="${link4_length/2} 0 0" rpy="0 0 0"/>
-        <mass value="0.3"/>
-        <inertia ixx="0.0005" ixy="0.0" ixz="0.0" iyy="0.001" iyz="0.0" izz="0.001"/>
-      </inertial>
-    </link>
-    <!-- Joint 5: Wrist pitch -->
-    <joint name="${prefix}joint5" type="revolute">
-      <parent link="${prefix}link4"/>
-      <child link="${prefix}link5"/>
-      <origin xyz="${link4_length} 0 0" rpy="0 0 0"/>
-      <axis xyz="0 1 0"/>
-      <limit lower="${-pi/2}" upper="${pi/2}" effort="${joint_effort_limit}" velocity="${joint_velocity_limit}"/>
-      <dynamics damping="${joint_damping}" friction="${joint_friction}"/>
-    </joint>
-    <!-- Link 5 -->
-    <link name="${prefix}link5">
-      <visual>
-        <origin xyz="${link5_length/2} 0 0" rpy="0 ${pi/2} 0"/>
-        <geometry>
-          <cylinder radius="${link_radius*0.6}" length="${link5_length}"/>
-        </geometry>
-        <material name="cyan">
-          <color rgba="0.2 0.8 0.8 1"/>
-        </material>
-      </visual>
-      <collision>
-        <origin xyz="${link5_length/2} 0 0" rpy="0 ${pi/2} 0"/>
-        <geometry>
-          <cylinder radius="${link_radius*0.6}" length="${link5_length}"/>
-        </geometry>
-      </collision>
-      <inertial>
-        <origin xyz="${link5_length/2} 0 0" rpy="0 0 0"/>
-        <mass value="0.2"/>
-        <inertia ixx="0.0002" ixy="0.0" ixz="0.0" iyy="0.0005" iyz="0.0" izz="0.0005"/>
-      </inertial>
-    </link>
-    <!-- Joint 6: Wrist roll (end effector) -->
-    <joint name="${prefix}joint6" type="revolute">
-      <parent link="${prefix}link5"/>
-      <child link="${prefix}link6"/>
-      <origin xyz="${link5_length} 0 0" rpy="0 0 0"/>
-      <axis xyz="1 0 0"/>
-      <limit lower="${-pi}" upper="${pi}" effort="${joint_effort_limit}" velocity="${joint_velocity_limit}"/>
-      <dynamics damping="${joint_damping}" friction="${joint_friction}"/>
-    </joint>
-    <!-- Link 6 (End effector) -->
-    <link name="${prefix}link6">
-      <visual>
-        <origin xyz="${link6_length/2} 0 0" rpy="0 ${pi/2} 0"/>
-        <geometry>
-          <cylinder radius="${link_radius*0.5}" length="${link6_length}"/>
-        </geometry>
-        <material name="magenta">
-          <color rgba="0.8 0.2 0.8 1"/>
-        </material>
-      </visual>
-      <collision>
-        <origin xyz="${link6_length/2} 0 0" rpy="0 ${pi/2} 0"/>
-        <geometry>
-          <cylinder radius="${link_radius*0.5}" length="${link6_length}"/>
-        </geometry>
-      </collision>
-      <inertial>
-        <origin xyz="${link6_length/2} 0 0" rpy="0 0 0"/>
-        <mass value="0.1"/>
-        <inertia ixx="0.0001" ixy="0.0" ixz="0.0" iyy="0.0002" iyz="0.0" izz="0.0002"/>
-      </inertial>
-    </link>
-    <!-- Tool center point (TCP) -->
-    <link name="${prefix}tcp"/>
-    <joint name="${prefix}tcp_joint" type="fixed">
-      <parent link="${prefix}link6"/>
-      <child link="${prefix}tcp"/>
-      <origin xyz="${link6_length} 0 0" rpy="0 0 0"/>
-    </joint>
+  <!-- material color setting -->
+  <material name="#ffffff">
+    <color rgba="1.000 1.000 1.000 1.0"/>
+  </material>
+  <joint name="base_link_to_floor_surface" type="fixed">
+    <origin xyz="0 0 0" rpy="0.0 0.0 0.0"/>
+    <parent link="${parent}"/>
+    <child link="floor_surface"/>
+  </joint>
+  <link name="floor_surface">
+    <inertial>
+      <origin xyz="1e-06 1.8e-05 -0.005002" rpy="0.0 0.0 0.0"/>
+      <mass value="0.000080925039"/>
+      <inertia ixx="0.00000013" ixy="-0" ixz="-0" iyy="0.00000013" iyz="0" izz="0.00000016"/>
+    </inertial>
+    <visual>
+      <origin xyz="0 0 0" rpy="0 0 0"/>
+      <geometry>
+        <mesh filename="package://mikata_arm_description/meshes/floor_surface.dae"/>
+      </geometry>
+      <material name="#ffffff"/>
+    </visual>
+  </link>
+  <joint name="floor_surface_to_Link1" type="fixed">
+    <origin xyz="0.0 0.0 0.0" rpy="0.0 0.0 0.0"/>
+    <parent link="floor_surface"/>
+    <child link="Link1"/>
+  </joint>
+  <link name="Link1">
+    <inertial>
+      <origin xyz="0.0 -0.0 0.021368" rpy="0.0 0.0 0.0"/>
+      <mass value="0.000001664356"/>
+      <inertia ixx="0" ixy="0" ixz="0" iyy="0" iyz="0" izz="0"/>
+    </inertial>
+    <visual>
+      <origin xyz="0 0 0" rpy="0 0 0"/>
+      <geometry>
+        <mesh filename="package://mikata_arm_description/meshes/Link1.dae"/>
+      </geometry>
+      <material name="#ffffff"/>
+    </visual>
+    <collision>
+      <origin xyz="0.0 0.0 0.015" rpy="0.0 0.0 0.0"/>
+      <geometry>
+        <cylinder radius="0.015" length="0.03"/>
+      </geometry>
+    </collision>
+  </link>
+  <joint name="joint1" type="revolute">
+    <origin xyz="0.0 0.0 0.03" rpy="0.0 0.0 0.0"/>
+    <axis xyz="0 0 1"/>
+    <parent link="Link1"/>
+    <child link="Link2"/>
+    <limit lower="-3.141592653589793" upper="3.141592653589793" effort="1.37" velocity="7.0"/>
+    <dynamics damping="0.18" friction="0.005"/>
+  </joint>
+  <gazebo reference="joint1">
+    <implicitSpringDamper>true</implicitSpringDamper>
+    <springStiffness>100</springStiffness>
+    <springReference>0.0</springReference>
+  </gazebo>
+  <link name="Link2">
+    <inertial>
+      <origin xyz="0.0 -0.0 0.107368" rpy="0.0 0.0 0.0"/>
+      <mass value="0.00000553095"/>
+      <inertia ixx="0.00000002" ixy="0" ixz="0" iyy="0.00000002" iyz="0" izz="0"/>
+    </inertial>
+    <visual>
+      <origin xyz="0 0 0" rpy="0 0 0"/>
+      <geometry>
+        <mesh filename="package://mikata_arm_description/meshes/Link2.dae"/>
+      </geometry>
+      <material name="#ffffff"/>
+    </visual>
+  </link>
+  <joint name="joint2" type="revolute">
+    <origin xyz="0.0 -0.0 0.076" rpy="0.0 0.0 0.0"/>
+    <axis xyz="0 1 0"/>
+    <parent link="Link2"/>
+    <child link="Link3"/>
+    <limit lower="-3.141592653589793" upper="3.141592653589793" effort="1.37" velocity="7.0"/>
+    <dynamics damping="0.18" friction="0.005"/>
+  </joint>
+  <gazebo reference="joint2">
+    <implicitSpringDamper>true</implicitSpringDamper>
+    <springStiffness>100</springStiffness>
+    <springReference>0.0</springReference>
+  </gazebo>
+  <link name="Link3">
+    <inertial>
+      <origin xyz="0.0 0.0 0.107368" rpy="0.0 0.0 0.0"/>
+      <mass value="0.000008777209"/>
+      <inertia ixx="0.00000004" ixy="0" ixz="-0" iyy="0.00000004" iyz="0" izz="0.00000002"/>
+    </inertial>
+    <visual>
+      <origin xyz="0 0 0" rpy="0 0 0"/>
+      <geometry>
+        <mesh filename="package://mikata_arm_description/meshes/Link3.dae"/>
+      </geometry>
+      <material name="#ffffff"/>
+    </visual>
+  </link>
+  <joint name="joint3" type="revolute">
+    <origin xyz="0.024 5e-05 0.168" rpy="0.0 0.0 0.0"/>
+    <axis xyz="0 1 0"/>
+    <parent link="Link3"/>
+    <child link="Link4"/>
+    <limit lower="-3.141592653589793" upper="3.141592653589793" effort="1.37" velocity="7.0"/>
+    <dynamics damping="0.18" friction="0.005"/>
+  </joint>
+  <gazebo reference="joint3">
+    <implicitSpringDamper>true</implicitSpringDamper>
+    <springStiffness>100</springStiffness>
+    <springReference>0.0</springReference>
+  </gazebo>
+  <link name="Link4">
+    <inertial>
+      <origin xyz="0.021909 -0.0 -0.0" rpy="0.0 0.0 0.0"/>
+      <mass value="0.000002893634"/>
+      <inertia ixx="0" ixy="0" ixz="0" iyy="0" iyz="0" izz="0"/>
+    </inertial>
+    <visual>
+      <origin xyz="0 0 0" rpy="0 0 0"/>
+      <geometry>
+        <mesh filename="package://mikata_arm_description/meshes/Link4.dae"/>
+      </geometry>
+      <material name="#ffffff"/>
+    </visual>
+  </link>
+  <joint name="joint4" type="revolute">
+    <origin xyz="0.045 0.0 0.0" rpy="0.0 0.0 0.0"/>
+    <axis xyz="1 0 0"/>
+    <parent link="Link4"/>
+    <child link="Link5"/>
+    <limit lower="-3.141592653589793" upper="3.141592653589793" effort="1.37" velocity="7.0"/>
+    <dynamics damping="0.18" friction="0.005"/>
+  </joint>
+  <gazebo reference="joint4">
+    <implicitSpringDamper>true</implicitSpringDamper>
+    <springStiffness>100</springStiffness>
+    <springReference>0.0</springReference>
+  </gazebo>
+  <link name="Link5">
+    <inertial>
+      <origin xyz="0.068461 -0.0 -0.0" rpy="0.0 0.0 0.0"/>
+      <mass value="0.000006380113"/>
+      <inertia ixx="0" ixy="0" ixz="0" iyy="0.00000001" iyz="0" izz="0.00000001"/>
+    </inertial>
+    <visual>
+      <origin xyz="0 0 0" rpy="0 0 0"/>
+      <geometry>
+        <mesh filename="package://mikata_arm_description/meshes/Link5.dae"/>
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
Commit message: ちゃんと動作してないがSetup Asssitantから生成したファイルを追加できた。

File: mikata_arm_description/urdf/mikata_arm.xacro (robot description, xacro)
@@ -76,4 +76,10 @@
       <material name="#ffffff"/>
     </visual>
+    <collision>
+      <origin xyz="0.0 0.0 0.0434" rpy="0.0 0.0 0.0"/>
+      <geometry>
+        <box size="0.02 0.02 0.0869"/>
+      </geometry>
+    </collision>
   </link>
   <joint name="joint2" type="revolute">
@@ -103,4 +109,10 @@
       <material name="#ffffff"/>
     </visual>
+    <collision>
+      <origin xyz="0.0145 0.0 0.0867" rpy="0.0 0.0 0.0"/>
+      <geometry>
+        <box size="0.04 0.03 0.19"/>
+      </geometry>
+    </collision>
   </link>
   <joint name="joint3" type="revolute">
@@ -130,4 +142,10 @@
       <material name="#ffffff"/>
     </visual>
+    <collision>
+      <origin xyz="0.02 0.0 0.0" rpy="0.0 0.0 0.0"/>
+      <geometry>
+        <box size="0.05 0.02 0.02"/>
+      </geometry>
+    </collision>
   </link>
   <joint name="joint4" type="revolute">
@@ -157,4 +175,10 @@
       <material name="#ffffff"/>
     </visual>
+    <collision>
+      <origin xyz="0.0585 0.0 0.0" rpy="0.0 0.0 0.0"/>
+      <geometry>
+        <box size="0.117 0.02 0.02"/>
+      </geometry>
+    </collision>
   </link>
   <joint name="joint5" type="revolute">
@@ -184,4 +208,10 @@
       <material name="#ffffff"/>
     </visual>
+    <collision>
+      <origin xyz="0.02 0.0 0.0" rpy="0.0 0.0 0.0"/>
+      <geometry>
+        <box size="0.05 0.02 0.02"/>
+      </geometry>
+    </collision>
   </link>
   <joint name="gripper_joint" type="revolute">
@@ -212,4 +242,10 @@
       <material name="#ffffff"/>
     </visual>
+    <collision>
+      <origin xyz="0.0275 -0.0012 -0.0035" rpy="0.0 0.0 0.0"/>
+      <geometry>
+        <box size="0.055 0.052 0.027"/>
+      </geometry>
+    </collision>
   </link>
   <joint name="gripper_sub1" type="revolute">
@@ -239,4 +275,10 @@
       <material name="#ffffff"/>
     </visual>
+    <collision>
+      <origin xyz="0.012 0.012 0.0" rpy="0.0 0.0 0.0"/>
+      <geometry>
+        <box size="0.034 0.034 0.012"/>
+      </geometry>
+    </collision>
   </link>
   <joint name="gripper_sub2" type="revolute">
@@ -266,4 +308,10 @@
       <material name="#ffffff"/>
     </visual>
+    <collision>
+      <origin xyz="0.012 -0.012 0.0" rpy="0.0 0.0 0.0"/>
+      <geometry>
+        <box size="0.034 0.034 0.012"/>
+      </geometry>
+    </collision>
   </link>
   </xacro:macro>

Commit message: ジョイントの制限を度からラジアンに変換し、各ジョイントの位置制限を設定

File: mikata_arm_description/urdf/mikata_arm.xacro (robot description, xacro)
@@ -2,4 +2,34 @@
 <robot xmlns:xacro="http://www.ros.org/wiki/xacro">
   <xacro:macro name="mikata_arm" params="prefix parent *origin">
+  <!-- ========================================== -->
+  <!-- Joint Limits Configuration (in degrees)    -->
+  <!-- ========================================== -->
+  <!-- Degree to Radian conversion -->
+  <xacro:property name="deg_to_rad" value="${pi/180.0}" />
+  <!-- Joint1: Position limits (degrees) -->
+  <xacro:property name="joint1_lower_deg" value="-175" />
+  <xacro:property name="joint1_upper_deg" value="175" />
+  <!-- Joint2: Position limits (degrees) -->
+  <xacro:property name="joint2_lower_deg" value="-145" />
+  <xacro:property name="joint2_upper_deg" value="90" />
+  <!-- Joint3: Position limits (degrees) -->
+  <xacro:property name="joint3_lower_deg" value="-80" />
+  <xacro:property name="joint3_upper_deg" value="90" />
+  <!-- Joint4: Position limits (degrees) -->
+  <xacro:property name="joint4_lower_deg" value="-175" />
+  <xacro:property name="joint4_upper_deg" value="175" />
+  <!-- Joint5: Position limits (degrees) -->
+  <xacro:property name="joint5_lower_deg" value="-110" />
+  <xacro:property name="joint5_upper_deg" value="100" />
+  <!-- Joint6: Position limits (degrees) -->
+  <xacro:property name="joint6_lower_deg" value="-175" />
+  <xacro:property name="joint6_upper_deg" value="175" />
+  <!-- Gripper joints: Position limits (degrees) -->
+  <xacro:property name="gripper_lower_deg" value="-45" />
+  <xacro:property name="gripper_upper_deg" value="45" />
+  <!-- Common properties for all joints -->
+  <xacro:property name="joint_effort" value="1.37" />
+  <xacro:property name="joint_velocity" value="7.0" />
+  <!-- ========================================== -->
   <!-- material color setting -->
   <material name="#ffffff">
@@ -55,5 +85,5 @@
     <parent link="Link1"/>
     <child link="Link2"/>
-    <limit lower="-3.141592653589793" upper="3.141592653589793" effort="1.37" velocity="7.0"/>
+    <limit lower="${joint1_lower_deg * deg_to_rad}" upper="${joint1_upper_deg * deg_to_rad}" effort="${joint_effort}" velocity="${joint_velocity}"/>
     <dynamics damping="0.18" friction="0.005"/>
   </joint>
@@ -88,5 +118,5 @@
     <parent link="Link2"/>
     <child link="Link3"/>
-    <limit lower="-3.141592653589793" upper="3.141592653589793" effort="1.37" velocity="7.0"/>
+    <limit lower="${joint2_lower_deg * deg_to_rad}" upper="${joint2_upper_deg * deg_to_rad}" effort="${joint_effort}" velocity="${joint_velocity}"/>
     <dynamics damping="0.18" friction="0.005"/>
   </joint>
@@ -121,5 +151,5 @@
     <parent link="Link3"/>
     <child link="Link4"/>
-    <limit lower="-3.141592653589793" upper="3.141592653589793" effort="1.37" velocity="7.0"/>
+    <limit lower="${joint3_lower_deg * deg_to_rad}" upper="${joint3_upper_deg * deg_to_rad}" effort="${joint_effort}" velocity="${joint_velocity}"/>
     <dynamics damping="0.18" friction="0.005"/>
   </joint>
@@ -154,5 +184,5 @@
     <parent link="Link4"/>
     <child link="Link5"/>
-    <limit lower="-3.141592653589793" upper="3.141592653589793" effort="1.37" velocity="7.0"/>
+    <limit lower="${joint4_lower_deg * deg_to_rad}" upper="${joint4_upper_deg * deg_to_rad}" effort="${joint_effort}" velocity="${joint_velocity}"/>
     <dynamics damping="0.18" friction="0.005"/>
   </joint>
@@ -187,5 +217,5 @@
     <parent link="Link5"/>
     <child link="Link6"/>
-    <limit lower="-3.141592653589793" upper="3.141592653589793" effort="1.37" velocity="7.0"/>
+    <limit lower="${joint5_lower_deg * deg_to_rad}" upper="${joint5_upper_deg * deg_to_rad}" effort="${joint_effort}" velocity="${joint_velocity}"/>
     <dynamics damping="0.18" friction="0.005"/>
   </joint>
@@ -220,5 +250,5 @@
     <parent link="Link6"/>
     <child link="gripper_base"/>
-    <limit lower="-3.141592653589793" upper="3.141592653589793" effort="1.37" velocity="7.0"/>
+    <limit lower="${joint6_lower_deg * deg_to_rad}" upper="${joint6_upper_deg * deg_to_rad}" effort="${joint_effort}" velocity="${joint_velocity}"/>
     <dynamics damping="0.18" friction="0.005"/>
   </joint>
@@ -254,5 +284,5 @@
     <parent link="gripper_base"/>
     <child link="gripper_link1"/>
-    <limit lower="-3.141592653589793" upper="3.141592653589793" effort="1.37" velocity="7.0"/>
+    <limit lower="${gripper_lower_deg * deg_to_rad}" upper="${gripper_upper_deg * deg_to_rad}" effort="${joint_effort}" velocity="${joint_velocity}"/>
     <dynamics damping="0.18" friction="0.005"/>
   </joint>
@@ -287,5 +317,5 @@
     <parent link="gripper_base"/>
     <child link="gripper_link2"/>
-    <limit lower="-3.141592653589793" upper="3.141592653589793" effort="1.37" velocity="7.0"/>
+    <limit lower="${gripper_lower_deg * deg_to_rad}" upper="${gripper_upper_deg * deg_to_rad}" effort="${joint_effort}" velocity="${joint_velocity}"/>
     <dynamics damping="0.18" friction="0.005"/>
   </joint>
