Commit message: グリッパーのジョイント設定を修正し、グリッパーのサブジョイントのミミックを追加

File: mikata_arm_description/urdf/mikata_arm.xacro (robot description, xacro)
@@ -319,4 +319,5 @@
     <limit lower="${gripper_lower_deg * deg_to_rad}" upper="${gripper_upper_deg * deg_to_rad}" effort="${joint_effort}" velocity="${joint_velocity}"/>
     <dynamics damping="0.18" friction="0.005"/>
+    <mimic joint="gripper_sub1" multiplier="-1.0" offset="0"/>
   </joint>
   <gazebo reference="gripper_sub2">

Commit message: RViz設定を更新し、表示オプションや衝突モデルの詳細を追加

File: mikata_arm_description/urdf/mikata_arm.xacro (robot description, xacro)
@@ -107,7 +107,7 @@
     </visual>
     <collision>
-      <origin xyz="0.0 0.0 0.0434" rpy="0.0 0.0 0.0"/>
-      <geometry>
-        <box size="0.02 0.02 0.0869"/>
+      <origin xyz="0.0 0.0 0.0284" rpy="0.0 0.0 0.0"/>
+      <geometry>
+        <cylinder radius="0.01" length="0.0569"/>
       </geometry>
     </collision>
@@ -140,7 +140,7 @@
     </visual>
     <collision>
-      <origin xyz="0.0145 0.0 0.0867" rpy="0.0 0.0 0.0"/>
-      <geometry>
-        <box size="0.04 0.03 0.19"/>
+      <origin xyz="0.0007 0.0 0.096" rpy="0.0 0.0 0.0"/>
+      <geometry>
+        <cylinder radius="0.006" length="0.15"/>
       </geometry>
     </collision>
@@ -173,7 +173,7 @@
     </visual>
     <collision>
-      <origin xyz="0.02 0.0 0.0" rpy="0.0 0.0 0.0"/>
-      <geometry>
-        <box size="0.05 0.02 0.02"/>
+      <origin xyz="0.0264 0.0 0.0" rpy="0.0 1.570796 0.0"/>
+      <geometry>
+        <cylinder radius="0.01" length="0.037"/>
       </geometry>
     </collision>
@@ -206,7 +206,7 @@
     </visual>
     <collision>
-      <origin xyz="0.0585 0.0 0.0" rpy="0.0 0.0 0.0"/>
-      <geometry>
-        <box size="0.117 0.02 0.02"/>
+      <origin xyz="0.04 0.0002 0.0" rpy="0.0 1.570796 0.0"/>
+      <geometry>
+        <cylinder radius="0.01" length="0.08"/>
       </geometry>
     </collision>
@@ -239,7 +239,7 @@
     </visual>
     <collision>
-      <origin xyz="0.02 0.0 0.0" rpy="0.0 0.0 0.0"/>
-      <geometry>
-        <box size="0.05 0.02 0.02"/>
+      <origin xyz="0.03 0.0 0.0" rpy="0.0 1.570796 0.0"/>
+      <geometry>
+        <cylinder radius="0.01" length="0.03"/>
       </geometry>
     </collision>
@@ -273,7 +273,7 @@
     </visual>
     <collision>
-      <origin xyz="0.0275 -0.0012 -0.0035" rpy="0.0 0.0 0.0"/>
-      <geometry>
-        <box size="0.055 0.052 0.027"/>
+      <origin xyz="0.0275 -0.0012 0.0045" rpy="0.0 0.0 0.0"/>
+      <geometry>
+        <box size="0.055 0.052 0.017"/>
       </geometry>
     </collision>
@@ -306,7 +306,7 @@
     </visual>
     <collision>
-      <origin xyz="0.012 0.012 0.0" rpy="0.0 0.0 0.0"/>
-      <geometry>
-        <box size="0.034 0.034 0.012"/>
+      <origin xyz="0.018 0.018 0.0001" rpy="-1.572037 0.000962 -0.781086"/>
+      <geometry>
+        <cylinder radius="0.0035" length="0.025"/>
       </geometry>
     </collision>
@@ -340,7 +340,7 @@
     </visual>
     <collision>
-      <origin xyz="0.012 -0.012 0.0" rpy="0.0 0.0 0.0"/>
-      <geometry>
-        <box size="0.034 0.034 0.012"/>
+      <origin xyz="0.018 -0.018 0.0" rpy="0.287266 1.569847 2.645491"/>
+      <geometry>
+        <cylinder radius="0.0035" length="0.025"/>
       </geometry>
     </collision>

Commit message: 各ジョイントの位置制限を設定 (#16)
* ジョイントの制限を度からラジアンに変換し、各ジョイントの位置制限を設定

* グリッパーのジョイント設定を修正し、グリッパーのサブジョイントのミミックを追加

* RViz設定を更新し、表示オプションや衝突モデルの詳細を追加

File: mikata_arm_description/urdf/mikata_arm.xacro (robot description, xacro)
@@ -2,4 +2,34 @@
 <robot xmlns:xacro="http://www.ros.org/wiki/xacro">
   <xacro:macro name="mikata_arm" params="prefix parent *origin">
+  <!-- ========================================== -->
+  <!-- Joint Limits Configuration (in degrees)    -->
+  <!-- ========================================== -->
+  <!-- Degree to Radian conversion -->
+  <xacro:property name="deg_to_rad" value="${pi/180.0}" />
+  <!-- Joint1: Position limits (degrees) -->
+  <xacro:property name="joint1_lower_deg" value="-175" />
+  <xacro:property name="joint1_upper_deg" value="175" />
+  <!-- Joint2: Position limits (degrees) -->
+  <xacro:property name="joint2_lower_deg" value="-145" />
+  <xacro:property name="joint2_upper_deg" value="90" />
+  <!-- Joint3: Position limits (degrees) -->
+  <xacro:property name="joint3_lower_deg" value="-80" />
+  <xacro:property name="joint3_upper_deg" value="90" />
+  <!-- Joint4: Position limits (degrees) -->
+  <xacro:property name="joint4_lower_deg" value="-175" />
+  <xacro:property name="joint4_upper_deg" value="175" />
+  <!-- Joint5: Position limits (degrees) -->
+  <xacro:property name="joint5_lower_deg" value="-110" />
+  <xacro:property name="joint5_upper_deg" value="100" />
+  <!-- Joint6: Position limits (degrees) -->
+  <xacro:property name="joint6_lower_deg" value="-175" />
+  <xacro:property name="joint6_upper_deg" value="175" />
+  <!-- Gripper joints: Position limits (degrees) -->
+  <xacro:property name="gripper_lower_deg" value="-45" />
+  <xacro:property name="gripper_upper_deg" value="45" />
+  <!-- Common properties for all joints -->
+  <xacro:property name="joint_effort" value="1.37" />
+  <xacro:property name="joint_velocity" value="7.0" />
+  <!-- ========================================== -->
   <!-- material color setting -->
   <material name="#ffffff">
@@ -55,5 +85,5 @@
     <parent link="Link1"/>
     <child link="Link2"/>
-    <limit lower="-3.141592653589793" upper="3.141592653589793" effort="1.37" velocity="7.0"/>
+    <limit lower="${joint1_lower_deg * deg_to_rad}" upper="${joint1_upper_deg * deg_to_rad}" effort="${joint_effort}" velocity="${joint_velocity}"/>
     <dynamics damping="0.18" friction="0.005"/>
   </joint>
@@ -77,7 +107,7 @@
     </visual>
     <collision>
-      <origin xyz="0.0 0.0 0.0434" rpy="0.0 0.0 0.0"/>
-      <geometry>
-        <box size="0.02 0.02 0.0869"/>
+      <origin xyz="0.0 0.0 0.0284" rpy="0.0 0.0 0.0"/>
+      <geometry>
+        <cylinder radius="0.01" length="0.0569"/>
       </geometry>
     </collision>
@@ -88,5 +118,5 @@
     <parent link="Link2"/>
     <child link="Link3"/>
-    <limit lower="-3.141592653589793" upper="3.141592653589793" effort="1.37" velocity="7.0"/>
+    <limit lower="${joint2_lower_deg * deg_to_rad}" upper="${joint2_upper_deg * deg_to_rad}" effort="${joint_effort}" velocity="${joint_velocity}"/>
     <dynamics damping="0.18" friction="0.005"/>
   </joint>
@@ -110,7 +140,7 @@
     </visual>
     <collision>
-      <origin xyz="0.0145 0.0 0.0867" rpy="0.0 0.0 0.0"/>
-      <geometry>
-        <box size="0.04 0.03 0.19"/>
+      <origin xyz="0.0007 0.0 0.096" rpy="0.0 0.0 0.0"/>
+      <geometry>
+        <cylinder radius="0.006" length="0.15"/>
       </geometry>
     </collision>
@@ -121,5 +151,5 @@
     <parent link="Link3"/>
     <child link="Link4"/>
-    <limit lower="-3.141592653589793" upper="3.141592653589793" effort="1.37" velocity="7.0"/>
+    <limit lower="${joint3_lower_deg * deg_to_rad}" upper="${joint3_upper_deg * deg_to_rad}" effort="${joint_effort}" velocity="${joint_velocity}"/>
     <dynamics damping="0.18" friction="0.005"/>
   </joint>
@@ -143,7 +173,7 @@
     </visual>
     <collision>
-      <origin xyz="0.02 0.0 0.0" rpy="0.0 0.0 0.0"/>
-      <geometry>
-        <box size="0.05 0.02 0.02"/>
+      <origin xyz="0.0264 0.0 0.0" rpy="0.0 1.570796 0.0"/>
+      <geometry>
+        <cylinder radius="0.01" length="0.037"/>
       </geometry>
     </collision>
@@ -154,5 +184,5 @@
     <parent link="Link4"/>
     <child link="Link5"/>
-    <limit lower="-3.141592653589793" upper="3.141592653589793" effort="1.37" velocity="7.0"/>
+    <limit lower="${joint4_lower_deg * deg_to_rad}" upper="${joint4_upper_deg * deg_to_rad}" effort="${joint_effort}" velocity="${joint_velocity}"/>
     <dynamics damping="0.18" friction="0.005"/>
   </joint>
@@ -176,7 +206,7 @@
     </visual>
     <collision>
-      <origin xyz="0.0585 0.0 0.0" rpy="0.0 0.0 0.0"/>
-      <geometry>
-        <box size="0.117 0.02 0.02"/>
+      <origin xyz="0.04 0.0002 0.0" rpy="0.0 1.570796 0.0"/>
+      <geometry>
+        <cylinder radius="0.01" length="0.08"/>
       </geometry>
     </collision>
@@ -187,5 +217,5 @@
     <parent link="Link5"/>
     <child link="Link6"/>
-    <limit lower="-3.141592653589793" upper="3.141592653589793" effort="1.37" velocity="7.0"/>
+    <limit lower="${joint5_lower_deg * deg_to_rad}" upper="${joint5_upper_deg * deg_to_rad}" effort="${joint_effort}" velocity="${joint_velocity}"/>
     <dynamics damping="0.18" friction="0.005"/>
   </joint>
@@ -209,7 +239,7 @@
     </visual>
     <collision>
-      <origin xyz="0.02 0.0 0.0" rpy="0.0 0.0 0.0"/>
-      <geometry>
-        <box size="0.05 0.02 0.02"/>
+      <origin xyz="0.03 0.0 0.0" rpy="0.0 1.570796 0.0"/>
+      <geometry>
+        <cylinder radius="0.01" length="0.03"/>
       </geometry>
     </collision>
@@ -220,5 +250,5 @@
     <parent link="Link6"/>
     <child link="gripper_base"/>
-    <limit lower="-3.141592653589793" upper="3.141592653589793" effort="1.37" velocity="7.0"/>
+    <limit lower="${joint6_lower_deg * deg_to_rad}" upper="${joint6_upper_deg * deg_to_rad}" effort="${joint_effort}" velocity="${joint_velocity}"/>
     <dynamics damping="0.18" friction="0.005"/>
   </joint>
@@ -243,7 +273,7 @@
     </visual>
     <collision>
-      <origin xyz="0.0275 -0.0012 -0.0035" rpy="0.0 0.0 0.0"/>
-      <geometry>
-        <box size="0.055 0.052 0.027"/>
+      <origin xyz="0.0275 -0.0012 0.0045" rpy="0.0 0.0 0.0"/>
+      <geometry>
+        <box size="0.055 0.052 0.017"/>
       </geometry>
     </collision>
@@ -254,5 +284,5 @@
     <parent link="gripper_base"/>
     <child link="gripper_link1"/>
-    <limit lower="-3.141592653589793" upper="3.141592653589793" effort="1.37" velocity="7.0"/>
+    <limit lower="${gripper_lower_deg * deg_to_rad}" upper="${gripper_upper_deg * deg_to_rad}" effort="${joint_effort}" velocity="${joint_velocity}"/>
     <dynamics damping="0.18" friction="0.005"/>
   </joint>
@@ -276,7 +306,7 @@
     </visual>
     <collision>
-      <origin xyz="0.012 0.012 0.0" rpy="0.0 0.0 0.0"/>
-      <geometry>
-        <box size="0.034 0.034 0.012"/>
+      <origin xyz="0.018 0.018 0.0001" rpy="-1.572037 0.000962 -0.781086"/>
+      <geometry>
+        <cylinder radius="0.0035" length="0.025"/>
       </geometry>
     </collision>
@@ -287,6 +317,7 @@
     <parent link="gripper_base"/>
     <child link="gripper_link2"/>
-    <limit lower="-3.141592653589793" upper="3.141592653589793" effort="1.37" velocity="7.0"/>
-    <dynamics damping="0.18" friction="0.005"/>
+    <limit lower="${gripper_lower_deg * deg_to_rad}" upper="${gripper_upper_deg * deg_to_rad}" effort="${joint_effort}" velocity="${joint_velocity}"/>
+    <dynamics damping="0.18" friction="0.005"/>
+    <mimic joint="gripper_sub1" multiplier="-1.0" offset="0"/>
   </joint>
   <gazebo reference="gripper_sub2">
@@ -309,7 +340,7 @@
     </visual>
     <collision>
-      <origin xyz="0.012 -0.012 0.0" rpy="0.0 0.0 0.0"/>
-      <geometry>
-        <box size="0.034 0.034 0.012"/>
+      <origin xyz="0.018 -0.018 0.0" rpy="0.287266 1.569847 2.645491"/>
+      <geometry>
+        <cylinder radius="0.0035" length="0.025"/>
       </geometry>
     </collision>
