Commit message: ハードウェア接続の設定を整理し、初期位置とコントローラー設定を新しい構成に移行

File: mikata_arm_description/urdf/mikata_arm.system.urdf.xacro (robot description, xacro)
@@ -2,8 +2,8 @@
 <robot xmlns:xacro="http://www.ros.org/wiki/xacro" name="mikata_arm">
   <xacro:arg name="prefix" default="" />
-  <xacro:arg name="initial_positions_file" default="$(find mikata_arm_bringup)/config/initial_positions.yaml" />
+  <xacro:arg name="initial_positions_file" default="$(find mikata_arm_description)/config/initial_positions.yaml" />
   <!-- Include robot model only (without ros2_control) -->
   <xacro:include filename="$(find mikata_arm_description)/urdf/mikata_arm.xacro" />
-  <xacro:include filename="$(find mikata_arm_description)/config/mikata_arm.ros2_control.xacro" />
+  <xacro:include filename="$(find mikata_arm_description)/urdf/mikata_arm.ros2_control.xacro" />
   <!-- Base link -->
   <link name="$(arg prefix)base_link" />

File: mikata_arm_description/urdf/mikata_arm.urdf.xacro (robot description, xacro)
@@ -5,5 +5,5 @@
   <xacro:include filename="$(find mikata_arm_description)/urdf/mikata_arm.xacro" />
   <!-- Import mikata_arm ros2_control description -->
-  <xacro:include filename="$(find mikata_arm_description)/config/mikata_arm.ros2_control.xacro" />
+  <xacro:include filename="$(find mikata_arm_description)/urdf/mikata_arm.ros2_control.xacro" />
   <link name="$(arg prefix)base_link" />
   <xacro:mikata_arm

File: mikata_arm_description/urdf/mikata_arm.xacro (robot description, xacro)
@@ -14,11 +14,11 @@
   <xacro:property name="joint2_upper_deg" value="90" />
   <!-- Joint3: Position limits (degrees) -->
-  <xacro:property name="joint3_lower_deg" value="-80" />
-  <xacro:property name="joint3_upper_deg" value="90" />
+  <xacro:property name="joint3_lower_deg" value="-90" />
+  <xacro:property name="joint3_upper_deg" value="80" />
   <!-- Joint4: Position limits (degrees) -->
   <xacro:property name="joint4_lower_deg" value="-175" />
   <xacro:property name="joint4_upper_deg" value="175" />
   <!-- Joint5: Position limits (degrees) -->
-  <xacro:property name="joint5_lower_deg" value="-110" />
+  <xacro:property name="joint5_lower_deg" value="-100" />
   <xacro:property name="joint5_upper_deg" value="100" />
   <!-- Joint6: Position limits (degrees) -->
