Commit message: ハードウェア接続の設定を追加 (#18)
* ハードウェア接続の設定を追加

* ハードウェア接続の設定を更新し、初期位置の定義を整理

* ハードウェア接続の設定を整理し、初期位置とコントローラー設定を新しい構成に移行

* ハードウェア接続の設定を更新し、フェイクハードウェアオプションを追加

* パッケージ設定を更新し、ライセンスをApache-2.0に変更。依存関係を整理し、説明を追加。

* 著者情報をpackage.xmlから削除

File: mikata_arm_description/urdf/mikata_arm.urdf.xacro (robot description, xacro)
@@ -2,17 +2,30 @@
 <!-- MikataArm 6-axis robot -->
 <robot xmlns:xacro="http://www.ros.org/wiki/xacro" name="mikata_arm">
+  <!-- Arguments -->
   <xacro:arg name="prefix" default="" />
+  <xacro:arg name="use_ros2_control" default="true" />
+  <xacro:arg name="use_fake_hardware" default="false" />
+  <xacro:arg name="initial_positions_file" default="$(find mikata_arm_description)/config/initial_positions.yaml" />
+  <!-- Include robot model -->
   <xacro:include filename="$(find mikata_arm_description)/urdf/mikata_arm.xacro" />
-  <!-- Import mikata_arm ros2_control description -->
-  <!-- <xacro:include filename="$(find mikata_arm_description)/ros2_control/mikata_arm.ros2_control.xacro" /> -->
+  <!-- Conditionally include ros2_control description -->
+  <xacro:if value="$(arg use_ros2_control)">
+    <xacro:include filename="$(find mikata_arm_description)/urdf/mikata_arm.ros2_control.xacro" />
+  </xacro:if>
+  <!-- Base link -->
   <link name="$(arg prefix)base_link" />
+  <!-- Robot arm -->
   <xacro:mikata_arm
       prefix="$(arg prefix)"
       parent="$(arg prefix)base_link">
-    <origin
-        xyz="0 0 0"
-        rpy="0 0 0" />
+    <origin xyz="0 0 0" rpy="0 0 0" />
   </xacro:mikata_arm>
-  <!-- <xacro:mikata_arm_ros2_control
-    name="mikata_arm" prefix="$(arg prefix)" /> -->
+  <!-- Conditionally add ros2_control hardware interface -->
+  <xacro:if value="$(arg use_ros2_control)">
+    <xacro:mikata_arm_ros2_control
+      name="mikata_arm"
+      prefix="$(arg prefix)"
+      use_fake_hardware="$(arg use_fake_hardware)"
+      initial_positions_file="$(arg initial_positions_file)" />
+  </xacro:if>
 </robot>

File: mikata_arm_description/urdf/mikata_arm.xacro (robot description, xacro)
@@ -14,11 +14,11 @@
   <xacro:property name="joint2_upper_deg" value="90" />
   <!-- Joint3: Position limits (degrees) -->
-  <xacro:property name="joint3_lower_deg" value="-80" />
-  <xacro:property name="joint3_upper_deg" value="90" />
+  <xacro:property name="joint3_lower_deg" value="-90" />
+  <xacro:property name="joint3_upper_deg" value="80" />
   <!-- Joint4: Position limits (degrees) -->
   <xacro:property name="joint4_lower_deg" value="-175" />
   <xacro:property name="joint4_upper_deg" value="175" />
   <!-- Joint5: Position limits (degrees) -->
-  <xacro:property name="joint5_lower_deg" value="-110" />
+  <xacro:property name="joint5_lower_deg" value="-100" />
   <xacro:property name="joint5_upper_deg" value="100" />
   <!-- Joint6: Position limits (degrees) -->
@@ -281,5 +281,5 @@
   <joint name="gripper_sub1" type="revolute">
     <origin xyz="0.045 0.0148 -0.011" rpy="0.0 0.0 0.0"/>
-    <axis xyz="0 0 1"/>
+    <axis xyz="0 0 -1"/>
     <parent link="gripper_base"/>
     <child link="gripper_link1"/>
@@ -314,5 +314,5 @@
   <joint name="gripper_sub2" type="revolute">
     <origin xyz="0.045 -0.0172 -0.011" rpy="0.0 0.0 0.0"/>
-    <axis xyz="0 0 1"/>
+    <axis xyz="0 0 -1"/>
     <parent link="gripper_base"/>
     <child link="gripper_link2"/>
