Commit message: ハードウェア接続の設定を更新し、フェイクハードウェアオプションを追加

File: mikata_arm_description/urdf/mikata_arm.ros2_control.xacro (robot description, xacro)
@@ -1,5 +1,5 @@
 <?xml version="1.0"?>
 <robot xmlns:xacro="http://www.ros.org/wiki/xacro">
-  <xacro:macro name="mikata_arm_ros2_control" params="name prefix:='' initial_positions_file:=''">
+  <xacro:macro name="mikata_arm_ros2_control" params="name prefix:='' use_fake_hardware:=false initial_positions_file:=''">
     <ros2_control name="${name}" type="system">
       <hardware>
@@ -7,5 +7,10 @@
         <param name="usb_port">/dev/ttyUSB0</param>
         <param name="baud_rate">1000000</param>
-        <param name="use_dummy">false</param>
+        <xacro:if value="${use_fake_hardware}">
+          <param name="use_dummy">true</param>
+        </xacro:if>
+        <xacro:unless value="${use_fake_hardware}">
+          <param name="use_dummy">false</param>
+        </xacro:unless>
         <xacro:if value="${initial_positions_file != ''}">
           <param name="initial_positions_file">${initial_positions_file}</param>

File: mikata_arm_description/urdf/mikata_arm.urdf.xacro (robot description, xacro)
@@ -2,17 +2,30 @@
 <!-- MikataArm 6-axis robot -->
 <robot xmlns:xacro="http://www.ros.org/wiki/xacro" name="mikata_arm">
+  <!-- Arguments -->
   <xacro:arg name="prefix" default="" />
+  <xacro:arg name="use_ros2_control" default="true" />
+  <xacro:arg name="use_fake_hardware" default="false" />
+  <xacro:arg name="initial_positions_file" default="$(find mikata_arm_description)/config/initial_positions.yaml" />
+  <!-- Include robot model -->
   <xacro:include filename="$(find mikata_arm_description)/urdf/mikata_arm.xacro" />
-  <!-- Import mikata_arm ros2_control description -->
-  <xacro:include filename="$(find mikata_arm_description)/urdf/mikata_arm.ros2_control.xacro" />
+  <!-- Conditionally include ros2_control description -->
+  <xacro:if value="$(arg use_ros2_control)">
+    <xacro:include filename="$(find mikata_arm_description)/urdf/mikata_arm.ros2_control.xacro" />
+  </xacro:if>
+  <!-- Base link -->
   <link name="$(arg prefix)base_link" />
+  <!-- Robot arm -->
   <xacro:mikata_arm
       prefix="$(arg prefix)"
       parent="$(arg prefix)base_link">
-    <origin
-        xyz="0 0 0"
-        rpy="0 0 0" />
+    <origin xyz="0 0 0" rpy="0 0 0" />
   </xacro:mikata_arm>
-  <xacro:mikata_arm_ros2_control
-    name="mikata_arm" prefix="$(arg prefix)" />
+  <!-- Conditionally add ros2_control hardware interface -->
+  <xacro:if value="$(arg use_ros2_control)">
+    <xacro:mikata_arm_ros2_control
+      name="mikata_arm"
+      prefix="$(arg prefix)"
+      use_fake_hardware="$(arg use_fake_hardware)"
+      initial_positions_file="$(arg initial_positions_file)" />
+  </xacro:if>
 </robot>

File: mikata_arm_moveit/config/mikata_arm.urdf.xacro (robot description, xacro)
@@ -1,5 +1,15 @@
 <?xml version="1.0"?>
 <robot xmlns:xacro="http://www.ros.org/wiki/xacro" name="mikata_arm">
-    <!-- Import mikata_arm urdf file -->
-    <xacro:include filename="$(find mikata_arm_description)/urdf/mikata_arm.urdf.xacro" />
+    <!-- MoveIt configuration: Robot model without ros2_control -->
+    <xacro:arg name="prefix" default="" />
+    <!-- Include robot model only -->
+    <xacro:include filename="$(find mikata_arm_description)/urdf/mikata_arm.xacro" />
+    <!-- Base link -->
+    <link name="$(arg prefix)base_link" />
+    <!-- Robot arm (without ros2_control for MoveIt) -->
+    <xacro:mikata_arm
+        prefix="$(arg prefix)"
+        parent="$(arg prefix)base_link">
+        <origin xyz="0 0 0" rpy="0 0 0" />
+    </xacro:mikata_arm>
 </robot>

Commit message: READMEとDockerfileの更新、USBポート設定の追加、Bashヒストリーにコマンドを追加

File: mikata_arm_description/urdf/mikata_arm.ros2_control.xacro (robot description, xacro)
@@ -1,9 +1,9 @@
 <?xml version="1.0"?>
 <robot xmlns:xacro="http://www.ros.org/wiki/xacro">
-  <xacro:macro name="mikata_arm_ros2_control" params="name prefix:='' use_fake_hardware:=false initial_positions_file:=''">
+  <xacro:macro name="mikata_arm_ros2_control" params="name prefix:='' use_fake_hardware:=false initial_positions_file:='' usb_port:=/dev/ttyUSB0">
     <ros2_control name="${name}" type="system">
       <hardware>
         <plugin>dynamixel_hardware/DynamixelHardware</plugin>
-        <param name="usb_port">/dev/ttyUSB0</param>
+        <param name="usb_port">${usb_port}</param>
         <param name="baud_rate">1000000</param>
         <xacro:if value="${use_fake_hardware}">

File: mikata_arm_description/urdf/mikata_arm.urdf.xacro (robot description, xacro)
@@ -7,4 +7,5 @@
   <xacro:arg name="use_fake_hardware" default="false" />
   <xacro:arg name="initial_positions_file" default="$(find mikata_arm_description)/config/initial_positions.yaml" />
+  <xacro:arg name="usb_port" default="/dev/ttyUSB0" />
   <!-- Include robot model -->
   <xacro:include filename="$(find mikata_arm_description)/urdf/mikata_arm.xacro" />
@@ -27,5 +28,6 @@
       prefix="$(arg prefix)"
       use_fake_hardware="$(arg use_fake_hardware)"
-      initial_positions_file="$(arg initial_positions_file)" />
+      initial_positions_file="$(arg initial_positions_file)"
+      usb_port="$(arg usb_port)" />
   </xacro:if>
 </robot>
